File: eagle/pendant2.brd (EAGLE design)
At the start: 10.2 x 29.8 mm, 7 parts, among them U1 TINY85-20-DIP

Commit message: fixing ICSP header
Parts:
- turned ICSP to 0 degrees
- renumbered SV1 to ICSP
Connections:
- net GND: now also ICSP.6; no longer ICSP.1
- net MISO: now also ICSP.1; no longer ICSP.3
- net MOSI: now also ICSP.4; no longer ICSP.6
- net RESET: now also ICSP.5; no longer ICSP.2
- net SCK: now also ICSP.3; no longer ICSP.4
- net VCC: now also ICSP.2; no longer ICSP.5
Routing:
- net MISO: track 16.2 -> 20.2 mm
- net VCC: track 7.40 -> 10.3 mm
- net MOSI: track 23.1 -> 25.3 mm
Changed lines of the file:
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@@
 <attribute name="NAME" x="3.81" y="6.35" size="1.27" layer="25" font="vector" ratio="10"/>
 </element>
-<element name="SV1" library="con-lstb" package="MA03-2" value="" x="5.08" y="12.7" smashed="yes" rot="R180">
-<attribute name="OC_NEWARK" value="unknown" x="5.08" y="12.7" size="1.778" layer="27" rot="R180" display="off"/>
-<attribute name="MPN" value="" x="5.08" y="12.7" size="1.778" layer="27" rot="R180" display="off"/>
-<attribute name="MF" value="" x="5.08" y="12.7" size="1.778" layer="27" rot="R180" display="off"/>
-<attribute name="OC_FARNELL" value="unknown" x="5.08" y="12.7" size="1.778" layer="27" rot="R180" display="off"/>
-<attribute name="NAME" x="7.62" y="9.779" size="1.27" layer="25" font="vector" ratio="10" rot="R180"/>
-<attribute name="VALUE" x="6.35" y="16.891" size="1.27" layer="27" ratio="10" rot="R180"/>
+<element name="ICSP" library="con-lstb" package="MA03-2" value="" x="5.08" y="12.7" smashed="yes">
+<attribute name="OC_NEWARK" value="unknown" x="5.08" y="12.7" size="1.778" layer="27" display="off"/>
+<attribute name="MPN" value="" x="5.08" y="12.7" size="1.778" layer="27" display="off"/>
+<attribute name="MF" value="" x="5.08" y="12.7" size="1.778" layer="27" display="off"/>
+<attribute name="OC_FARNELL" value="unknown" x="5.08" y="12.7" size="1.778" layer="27" display="off"/>
+<attribute name="NAME" x="3.175" y="8.636" size="1.27" layer="25" font="vector" ratio="10"/>
+<attribute name="VALUE" x="3.81" y="8.509" size="1.27" layer="27" ratio="10"/>
 </element>
 <element name="U1" library="SparkFun-DigitalIC" package="DIP08" value="TINY85-20-DIP" x="5.08" y="20.32" smashed="yes" rot="R180">
@@
 <signal name="VCC">
 <contactref element="U1" pad="8"/>
-<contactref element="SV1" pad="5"/>
-<wire x1="2.54" y1="13.97" x2="3.81" y2="15.24" width="0.4064" layer="1"/>
-<wire x1="3.81" y1="15.24" x2="7.62" y2="15.24" width="0.4064" layer="1"/>
-<wire x1="7.62" y1="15.24" x2="8.89" y2="16.51" width="0.4064" layer="1"/>
+<contactref element="ICSP" pad="2"/>
+<wire x1="2.54" y1="13.97" x2="3.81" y2="12.7" width="0.4064" layer="1"/>
+<wire x1="3.81" y1="12.7" x2="8.255" y2="12.7" width="0.4064" layer="1"/>
+<wire x1="8.255" y1="12.7" x2="8.89" y2="13.335" width="0.4064" layer="1"/>
+<wire x1="8.89" y1="13.335" x2="8.89" y2="16.51" width="0.4064" layer="1"/>
 </signal>
 <signal name="GND">
 <contactref element="D1" pad="2"/>
-<contactref element="SV1" pad="1"/>
+<contactref element="ICSP" pad="6"/>
 <contactref element="S1" pad="2"/>
 <polygon width="0.254" layer="16" isolate="0.254">
@@
 </signal>
 <signal name="RESET">
-<contactref element="SV1" pad="2"/>
+<contactref element="ICSP" pad="5"/>
 <contactref element="U1" pad="1"/>
 <wire x1="7.62" y1="11.43" x2="8.89" y2="12.7" width="0.4064" layer="16"/>
@@
 <signal name="MOSI">
 <contactref element="U1" pad="5"/>
-<contactref element="SV1" pad="6"/>
 <contactref element="R1" pad="1"/>
-<wire x1="1.27" y1="16.51" x2="1.27" y2="12.7" width="0.4064" layer="16"/>
-<wire x1="1.27" y1="12.7" x2="2.54" y2="11.43" width="0.4064" layer="16"/>
+<wire x1="1.27" y1="16.51" x2="1.27" y2="13.335" width="0.4064" layer="16"/>
 <wire x1="7.62" y1="26.67" x2="6.35" y2="27.94" width="0.4064" layer="16"/>
 <wire x1="6.35" y1="27.94" x2="4.445" y2="27.94" width="0.4064" layer="16"/>
@@
 <wire x1="5.08" y1="24.765" x2="5.08" y2="20.32" width="0.4064" layer="16"/>
 <wire x1="5.08" y1="20.32" x2="1.27" y2="16.51" width="0.4064" layer="16"/>
+<contactref element="ICSP" pad="4"/>
+<wire x1="5.08" y1="13.97" x2="3.81" y2="12.7" width="0.4064" layer="16"/>
+<wire x1="3.81" y1="12.7" x2="1.905" y2="12.7" width="0.4064" layer="16"/>
+<wire x1="1.905" y1="12.7" x2="1.27" y2="13.335" width="0.4064" layer="16"/>
 </signal>
 <signal name="MISO">
 <contactref element="U1" pad="6"/>
 <contactref element="R2" pad="1"/>
-<contactref element="SV1" pad="3"/>
-<wire x1="5.08" y1="13.97" x2="3.81" y2="15.24" width="0.4064" layer="16"/>
-<wire x1="3.81" y1="15.24" x2="3.81" y2="16.51" width="0.4064" layer="16"/>
 <wire x1="3.81" y1="16.51" x2="3.81" y2="17.145" width="0.4064" layer="16"/>
 <wire x1="3.81" y1="17.145" x2="7.62" y2="20.955" width="0.4064" layer="16"/>
@@
 <wire x1="7.62" y1="24.765" x2="5.715" y2="26.67" width="0.4064" layer="16"/>
 <wire x1="5.715" y1="26.67" x2="5.08" y2="26.67" width="0.4064" layer="16"/>
+<contactref element="ICSP" pad="1"/>
+<wire x1="3.81" y1="16.51" x2="2.54" y2="15.24" width="0.4064" layer="1"/>
+<wire x1="2.54" y1="15.24" x2="1.905" y2="15.24" width="0.4064" layer="1"/>
+<wire x1="1.905" y1="15.24" x2="1.27" y2="14.605" width="0.4064" layer="1"/>
+<wire x1="1.27" y1="14.605" x2="1.27" y2="12.7" width="0.4064" layer="1"/>
+<wire x1="1.27" y1="12.7" x2="2.54" y2="11.43" width="0.4064" layer="1"/>
 </signal>
 <signal name="SCK">
 <contactref element="U1" pad="7"/>
-<contactref element="SV1" pad="4"/>
+<contactref element="ICSP" pad="3"/>
 <contactref element="S1" pad="1"/>
 <wire x1="5.08" y1="11.43" x2="6.35" y2="12.7" width="0.4064" layer="16"/>
